File: kicad/lm386-audio.kicad_pcb (KiCad board)
At the start: 4 copper layers, 70.5 x 53 mm, 31 parts, among them J3 Gain, J4 Audio_IN, J6 Headphones, Q1 AO3407, U1 LM386, U2 SD6271 Step Up

Commit message: clean up + documentation
Parts:
- added G***: LOGO, LOGO, F.Cu at (182.6, 51.7)
Routing:
- net Net-(D2-K): track 14.6 -> 31.1 mm
- net GND: track 164.8 -> 168.2 mm, vias 0 -> 1
- net +12V: track 133.1 -> 131.9 mm
Other:
- board text added: "BAT+"
- board text added: "BAT-"
- board text removed: "OLD_OUT"
